File: hardware/leds/led.kicad_pcb (KiCad board)
At the start: 2 copper layers, 75 parts, among them P1 ICD3 header, U1 PIC18F2450, U2 74HC594, U3 74HC594, U4 74HC594, U5 74HC594, X1 20 MHz

Commit message: leds on the edge. routing not quite done yet
Parts:
- added P2: ICD3 header, Pin_Header_Straight_1x06, F.Cu at (135.9, 30.5)
- moved U5 106.0 mm to (163.8, 120.7)
- moved R19 100.6 mm to (135.9, 111.8)
- moved R20 100.6 mm to (135.9, 114.3)
- moved R21 100.6 mm to (135.9, 116.8)
- moved R22 100.6 mm to (135.9, 119.4)
- moved R23 100.6 mm to (135.9, 121.9)
- moved R24 100.6 mm to (135.9, 124.5)
- moved R25 100.6 mm to (135.9, 127.0)
- moved R26 100.6 mm to (135.9, 129.5)
- moved R10 99.6 mm to (135.9, 88.9)
- moved R3 99.6 mm to (135.9, 71.1)
- moved R4 99.6 mm to (135.9, 73.7)
- moved R5 99.6 mm to (135.9, 76.2)
- moved R6 99.6 mm to (135.9, 78.7)
- moved R7 99.6 mm to (135.9, 81.3)
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Connections:
- R1 pad 1: Net-(R1-Pad1) -> Net-(P1-Pad1)
- U1 pad 1: Net-(R1-Pad1) -> Net-(P1-Pad1)
- U1 pad 26: Net-(P1-Pad4) -> Net-(P1-Pad6)
- U1 pad 28: Net-(P1-Pad6) -> Net-(P1-Pad4)
Routing:
- net GND: track 0.00 -> 393.8 mm
- net +5V: track 0.00 -> 332.5 mm, vias 0 -> 6
- net Net-(U1-Pad6): track 0.00 -> 159.3 mm, vias 0 -> 3
- net Net-(U1-Pad7): track 0.00 -> 155.6 mm
- net Net-(D25-Pad1): track 0.00 -> 124.6 mm
- net Net-(D26-Pad1): track 0.00 -> 121.0 mm
- net Net-(D27-Pad1): track 0.00 -> 117.4 mm
- net Net-(D28-Pad1): track 0.00 -> 113.8 mm
- net Net-(D29-Pad1): track 0.00 -> 110.2 mm
- net Net-(D30-Pad1): track 0.00 -> 106.6 mm
- net Net-(D31-Pad1): track 0.00 -> 103.4 mm
- net Net-(D32-Pad1): track 0.00 -> 99.4 mm
- net Net-(D1-Pad1): track 0.00 -> 95.8 mm
- net Net-(P1-Pad1): track 0.00 -> 94.8 mm
- net Net-(D2-Pad1): track 0.00 -> 92.2 mm
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- added copper zone on F.Cu, net +5V
- added copper zone on B.Cu, net GND

Commit message: not sure
Routing:
- net Net-(R11-Pad2): track 0.00 -> 38.5 mm
- net Net-(R27-Pad2): track 0.00 -> 37.4 mm
- net Net-(R19-Pad2): track 7.18 -> 40.1 mm
- net Net-(R23-Pad2): track 0.00 -> 30.4 mm
- net Net-(R25-Pad2): track 0.00 -> 30.4 mm
- net Net-(R24-Pad2): track 0.00 -> 30.4 mm
- net Net-(R22-Pad2): track 0.00 -> 30.4 mm
- net Net-(R21-Pad2): track 0.00 -> 30.4 mm
- net Net-(R20-Pad2): track 0.00 -> 30.4 mm
- net Net-(R26-Pad2): track 0.00 -> 30.4 mm
- net Net-(R3-Pad2): track 7.18 -> 36.9 mm
- net Net-(R16-Pad2): track 0.00 -> 28.8 mm
- net Net-(R18-Pad2): track 0.00 -> 28.8 mm
- net Net-(R17-Pad2): track 0.00 -> 28.8 mm
- net Net-(R15-Pad2): track 0.00 -> 28.8 mm
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
Commit message: More compact design
Parts:
- removed P2: ICD3 header, Pin_Header_Straight_1x06
- moved U2 53.5 mm to (114.3, 68.6), turned to 90 degrees
- moved R26 45.5 mm to (109.2, 92.7), turned to 270 degrees
- moved P1 44.2 mm to (212.7, 66.0), turned to 0 degrees
- moved R25 41.9 mm to (111.8, 92.7), turned to 270 degrees
- moved U5 39.5 mm to (130.8, 99.1), turned to 270 degrees
- moved R24 38.4 mm to (114.3, 92.7), turned to 270 degrees
- moved R23 34.9 mm to (116.8, 92.7), turned to 270 degrees
- moved R27 32.4 mm to (114.3, 74.9), turned to 90 degrees
- moved R22 31.4 mm to (119.4, 92.7), turned to 270 degrees
- moved R28 28.8 mm to (116.8, 74.9), turned to 90 degrees
- moved R2 28.2 mm to (204.5, 72.4), turned to 0 degrees
- moved R21 27.9 mm to (121.9, 92.7), turned to 270 degrees
- moved R10 25.7 mm to (157.5, 74.9), turned to 90 degrees
- moved U3 25.7 mm to (138.4, 68.6), turned to 90 degrees
- moved R29 25.2 mm to (119.4, 74.9), turned to 90 degrees
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Connections:
- U2 pad 16: VCC -> +5V
- U3 pad 16: VCC -> +5V
- U4 pad 16: VCC -> +5V
- U5 pad 16: VCC -> +5V
Routing:
- net VCC: track 81.4 -> 0.00 mm
- net Net-(P1-Pad1): track 94.8 -> 23.4 mm
- net Net-(D24-Pad1): track 63.1 -> 5.08 mm
- net Net-(U1-Pad7): track 155.6 -> 207.6 mm, vias 0 -> 5
- net Net-(D23-Pad1): track 64.3 -> 15.1 mm
- net Net-(D22-Pad1): track 65.6 -> 19.6 mm
- net Net-(D21-Pad1): track 65.2 -> 25.6 mm
- net Net-(U1-Pad6): track 159.3 -> 198.7 mm, vias 3 -> 5
- net Net-(U1-Pad2): track 52.6 -> 91.0 mm
- net +5V: track 332.5 -> 296.2 mm, vias 6 -> 4
- net Net-(D20-Pad1): track 66.5 -> 30.6 mm
- net Net-(P1-Pad4): track 43.0 -> 8.31 mm
- net Net-(D25-Pad1): track 124.6 -> 91.2 mm
- net Net-(D26-Pad1): track 121.0 -> 90.1 mm
- net Net-(P1-Pad6): track 38.7 -> 8.31 mm
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